File: TFRAS/TFRAS_TOP/TFRAS_TOP.kicad_pcb (KiCad board)
At the start: 4 copper layers, 24 x 24 mm, 27 parts, among them J1 Molex 555600807, J2 Molex 555600807, U1 ATmega328PB-MU, U2 MCP1754S-3302xCB, U3 MAX14783EATA+T, U4 74HC4067BQ,118, U5 74HC4067BQ,118, U6 74HC4067BQ,118, U7 74HC4067BQ,118, U8 74HC4067BQ,118, U9 74HC4067BQ,118, Y1 Resonator

Commit message: organization and updating project files
Parts:
- removed D1: CDSOT23-SM712, Package_TO_SOT_SMD:SOT-23
- removed D2: 1N4148, Diode_SMD:D_0402_1005Metric
- removed J2: Molex 555600807, Connector_Molex:Molex_SlimStack_55560-0801_2x40_P0.50mm_Vertical
- removed U6, U7, U8, U9: 74HC4067BQ,118, 74LVCH8T245BQQ10J
- removed Y1: Resonator, Crystal:Resonator_SMD_muRata_CSTxExxV-3Pin_3.0x1.1mm
- added C7: 100nF, Capacitor_SMD:C_0402_1005Metric, B.Cu at (33.7, 22.3)
- added C8: 100nF, Capacitor_SMD:C_0402_1005Metric, B.Cu at (32.7, 41.2)
- added G***: LOGO, Rare flowers:TFRAS, B.Cu at (28.4, 24.3)
- added J3: UPDI-POGO, Connector:Tag-Connect_TC2030-IDC-NL_2x03_P1.27mm_Vertical, F.Cu at (42.0, 30.1)
- added J4: TOP, Connector_FFC-FPC:Molex_200528-0170_1x17-1MP_P1.00mm_Horizontal, F.Cu at (32.0, 24.2)
- added JPWR1: Conn_01x02_Female, Connector_PinHeader_1.27mm:PinHeader_1x02_P1.27mm_Vertical, B.Cu at (41.3, 34.1)
- added R5: 10k, Resistor_SMD:R_0402_1005Metric, B.Cu at (32.7, 30.7)
- added R7: 10k, Resistor_SMD:R_0402_1005Metric, B.Cu at (36.1, 36.4)
- added R8: RTERM, Resistor_SMD:R_0805_2012Metric_Pad1.20x1.40mm_HandSolder, F.Cu at (23.5, 33.2)
- added RS4851: Conn_01x02_Female, Connector_PinHeader_1.27mm:PinHeader_1x02_P1.27mm_Vertical, B.Cu at (23.3, 35.5)
- added RST1: TestPoint_Small, TestPoint:TestPoint_Pad_1.0x1.0mm, B.Cu at (31.1, 29.9)
- C1: value 1uF/16V -> 10u; footprint Capacitor_SMD:C_0402_1005Metric -> Capacitor_SMD:C_1206_3216Metric; moved to B.Cu
- C2: value 1uF/6.3V -> 100u; footprint Capacitor_SMD:C_0402_1005Metric -> Capacitor_SMD:C_1206_3216Metric; moved to B.Cu
- C3, C5, C6, L1: moved to B.Cu
- J1: value Molex 555600807 -> BOTTOM; footprint Connector_Molex:Molex_SlimStack_55560-0801_2x40_P0.50mm_Vertical -> Connector_FFC-FPC:Molex_200528-0170_1x17-1MP_P1.00mm_Horizontal; moved to F.Cu
- R1, R2: value 10K -> 10k
- R3, R4: footprint Resistor_SMD:R_0603_1608Metric -> Resistor_SMD:R_1206_3216Metric; moved to B.Cu
- R6: value 10K -> 10k; moved to B.Cu
- U1: value ATmega328PB-MU -> ATmega4809-A; footprint Package_DFN_QFN:QFN-32-1EP_5x5mm_P0.5mm_EP3.1x3.1mm -> Package_QFP:TQFP-48_7x7mm_P0.5mm
- U2: value MCP1754S-3302xCB -> AMS1117-3.3; footprint Package_TO_SOT_SMD:SOT-23 -> Package_TO_SOT_SMD:SOT-223-3_TabPin2; moved to B.Cu
- U3: value MAX14783EATA+T -> SN65HVD75; footprint Package_DFN_QFN:DFN-8_2x2mm_P0.5mm -> Package_SO:SOIC-8_3.9x4.9mm_P1.27mm; moved to B.Cu
- U4, U5: value 74HC4067BQ,118 -> 74HCT4051; footprint 74LVCH8T245BQQ10J -> Rare flowers:SOT763-1(DHVQFN16)
- moved U5 38.2 mm to (28.7, 41.5), turned to 90 degrees
- moved U2 25.5 mm to (40.3, 39.5), turned to 270 degrees
- moved R3 24.7 mm to (21.3, 37.2)
- moved U4 24.1 mm to (37.7, 22.4), turned to 270 degrees
- moved U3 20.6 mm to (23.9, 31.7), turned to 180 degrees
- moved R4 19.8 mm to (25.4, 37.1)
- moved C1 19.7 mm to (41.4, 30.7), turned to 180 degrees
- moved C6 19.4 mm to (21.7, 28.4), turned to 180 degrees
- moved C2 18.4 mm to (37.6, 33.7), turned to 0 degrees
- moved C4 14.4 mm to (38.0, 33.2)
- moved C3 14.4 mm to (28.9, 36.5), turned to 270 degrees
- moved R1 13.7 mm to (38.7, 36.0), turned to 180 degrees
- moved TH1 12.7 mm to (38.6, 35.0), turned to 0 degrees
- moved L1 10.7 mm to (32.5, 35.1)
- moved R6 10.7 mm to (32.7, 32.6)
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Connections:
- C4 pad 1: +3V3 -> Net-(C3-Pad1)
- C5 pad 1: Net-(C5-Pad1) -> Net-(C3-Pad1)
- J1 pad 1: BS17 -> G-
- J1 pad 10: BS12 -> GND
- J1 pad 11: Net-(J1-Pad11) -> Vin
- J1 pad 12: BS11 -> H-
- J1 pad 13: GND -> I-
- J1 pad 14: BS10 -> J-
- J1 pad 15: GND -> K-
- J1 pad 16: BS9 -> L-
- J1 pad 17: GND -> M-
- J1 pad 2: BS18 -> F-
- J1 pad 3: BS15 -> E-
- J1 pad 4: BS16 -> D-
- J1 pad 5: Vin -> C-
- J1 pad 6: BS14 -> B-
- J1 pad 7: Vin -> RS485_A-
- J1 pad 8: BS13 -> RS485_B+
- J1 pad 9: Vin -> A-
- L1 pad 2: Net-(C5-Pad1) -> Net-(C3-Pad1)
- R1 pad 2: ADC -> ADC_THERM
- R2 pad 1: Net-(D2-Pad1) -> A_TOP
- R2 pad 2: RST -> GND
- R6 pad 1: GND -> Net-(C3-Pad1)
- R6 pad 2: Z -> Net-(R5-Pad1)
- TH1 pad 1: ADC -> ADC_THERM
- U1 pad 1: S0 -> K
- U1 pad 10: E2 -> S2-
- U1 pad 11: E3 -> S1-
- U1 pad 12: E4 -> S0-
- U1 pad 13: E5 -> B-
- U1 pad 14: E6 -> Net-(C3-Pad1)
- U1 pad 15: MOSI -> GND
- U1 pad 16: MISO -> Net-(U1-Pad16)
- U1 pad 17: SCK -> Net-(U1-Pad17)
- U1 pad 18: Net-(C5-Pad1) -> Net-(U1-Pad18)
- U1 pad 2: S1 -> M
- U1 pad 20: Net-(C3-Pad1) -> Net-(U1-Pad20)
- U1 pad 21: GND -> Net-(U1-Pad21)
- U1 pad 23: ADC -> A_BOTTOM
- U1 pad 24: Z -> H-
- U1 pad 25: Net-(U1-Pad25) -> J-
- U1 pad 26: Net-(U1-Pad26) -> L-
- U1 pad 27: Net-(U1-Pad27) -> ADC_THERM
- U1 pad 28: Net-(U1-Pad28) -> Net-(C3-Pad1)
- U1 pad 29: RST -> GND
- U1 pad 3: S2 -> Net-(U1-Pad3)
- U1 pad 30: UART_RX -> Net-(U1-Pad30)
- U1 pad 31: UART_TX -> S2
- U1 pad 32: RS485_EN -> S1
- U1 pad 33: GND -> S0
- U1 pad 4: +3V3 -> Net-(U1-Pad4)
- U1 pad 5: GND -> Net-(U1-Pad5)
- U1 pad 6: S3 -> Net-(U1-Pad6)
- U1 pad 7: Net-(U1-Pad7) -> F-
- U1 pad 8: Net-(U1-Pad8) -> D-
- U1 pad 9: E1 -> Net-(U1-Pad9)
- U3 pad 6: Net-(R4-Pad2) -> Net-(R3-Pad2)
- U3 pad 7: Net-(R3-Pad2) -> Net-(R4-Pad2)
- U4 pad 1: +3V3 -> L
- U4 pad 10: S0 -> S1
- U4 pad 11: S1 -> S0
- U4 pad 12: GND -> D
- U4 pad 13: S3 -> B
- U4 pad 14: S2 -> H
- U4 pad 15: E1 -> J
- U4 pad 16: BS15 -> +3V3
- U4 pad 2: BS9 -> Net-(U4-Pad2)
- U4 pad 3: BS10 -> A_TOP
- U4 pad 4: BS11 -> Net-(U4-Pad4)
- U4 pad 5: BS12 -> F
- U4 pad 6: BS13 -> GND
- U4 pad 7: BS14 -> GND
- U4 pad 8: BS16 -> GND
- U4 pad 9: BS18 -> S2
- U5 pad 1: +3V3 -> C-
- U5 pad 10: S0 -> S1-
- U5 pad 11: S1 -> S0-
- U5 pad 12: GND -> A-
- U5 pad 13: S3 -> I-
- U5 pad 14: S2 -> K-
- U5 pad 15: E3 -> M-
- U5 pad 16: BS31 -> +3V3
- U5 pad 2: BS23 -> Net-(U5-Pad2)
- U5 pad 3: BS22 -> A_BOTTOM
- U5 pad 4: BS21 -> E-
- U5 pad 5: BS20 -> G-
- U5 pad 6: BS19 -> GND
- U5 pad 7: BS18 -> GND
- U5 pad 8: BS17 -> GND
- U5 pad 9: BS16 -> S2-
Routing:
- net RS485_B+: track 5.93 -> 39.6 mm, vias 1 -> 2
- net Vin: track 5.87 -> 32.6 mm, vias 1 -> 2
- net RS485_A-: track 6.48 -> 33.1 mm, vias 1 -> 2
- net +3V3: track 62.2 -> 36.4 mm, vias 5 -> 8
- net Net-(C3-Pad1): track 2.74 -> 23.4 mm, vias 0 -> 3
- net A_BOTTOM: track 0.00 -> 17.6 mm, vias 0 -> 1
- net A_TOP: track 0.00 -> 16.9 mm, vias 0 -> 1
- net C-: track 0.00 -> 15.3 mm, vias 0 -> 1
- net I-: track 0.00 -> 14.5 mm, vias 0 -> 2
- net L: track 0.00 -> 14.2 mm, vias 0 -> 1
- net RST: track 14.0 -> 0.00 mm, vias 2 -> 0
- net E-: track 0.00 -> 13.4 mm, vias 0 -> 1
- net UPDI: track 0.00 -> 13.2 mm
- net M-: track 0.00 -> 12.6 mm, vias 0 -> 1
- net G-: track 0.00 -> 12.4 mm, vias 0 -> 3
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- added copper zone on In2.Cu, net +3V3
- added copper zone on B.Cu, net GND
- added copper zone on F.Cu, net GND
- added copper zone on In1.Cu, net GND
Other:
- net class Default: clearance 0.2 -> 0.15; via_dia 0.8 -> 0.6
- rule trace_clearance: 0.2 -> 0.15
- rule trace_min: 0.2 -> 0.09
- rule via_min_drill: 0.3 -> 0.2
- board text added: "A"
- board text added: "B"
- board text added: "REV 0"
- board text added: "Rt"
- board text added: "V+"
- board text added: "V-"
