File: TFRAS/TFRAS_TOP/TFRAS_TOP.sch (KiCad schematic (older format))
At the start: 27 parts, among them J1 Molex 555600807, J2 Molex 555600807, U1 ATmega328PB-MU, U2 MCP1754S-3302xCB, U3 MAX14783EATA+T, U4 74HC4067BQ,118, U5 74HC4067BQ,118, U6 74HC4067BQ,118, U7 74HC4067BQ,118, U8 74HC4067BQ,118, U9 74HC4067BQ,118, Y1 Resonator

Commit message: organization and updating project files
Parts:
- removed D1: CDSOT23-SM712, Package_TO_SOT_SMD:SOT-23, symbol Power_Protection:SP0502BAHT
- removed D2: 1N4148, Diode_SMD:D_0402_1005Metric, symbol Diode:1N4148
- removed J1, J2: Molex 555600807, Connector_Molex:Molex_SlimStack_55560-0801_2x40_P0.50mm_Vertical, symbol Connector_Generic:Conn_02x40_Odd_Even
- removed U1: ATmega328PB-MU, Package_DFN_QFN:QFN-32-1EP_5x5mm_P0.5mm_EP3.1x3.1mm, symbol MCU_Microchip_ATmega:ATmega328PB-MU
- removed U2: MCP1754S-3302xCB, Package_TO_SOT_SMD:SOT-23, symbol Regulator_Linear:MCP1754S-3302xCB
- removed U3: MAX14783EATA+T, Package_DFN_QFN:DFN-8_2x2mm_P0.5mm, symbol Interface_UART:MAX485E
- removed U4, U5, U6, U7, U8, U9: 74HC4067BQ,118, 74LVCH8T245BQQ10J, symbol 74HC4067BQ_118:74HC4067BQ,118
- removed Y1: Resonator, Crystal:Resonator_SMD_muRata_CSTxExxV-3Pin_3.0x1.1mm, symbol Device:Resonator_Small
- added C7, C8: 100nF, Capacitor_SMD:C_0402_1005Metric, symbol Device:C
- added J1: BOTTOM, Connector_FFC-FPC:Molex_200528-0170_1x17-1MP_P1.00mm_Horizontal, symbol Connector:Conn_01x17_Male
- added J3: UPDI-POGO, Connector:Tag-Connect_TC2030-IDC-NL_2x03_P1.27mm_Vertical, symbol Connector:AVR-ISP-6
- added J4: TOP, Connector_FFC-FPC:Molex_200528-0170_1x17-1MP_P1.00mm_Horizontal, symbol Connector:Conn_01x17_Male
- added JPWR1, RS4851: Conn_01x02_Female, Connector_PinHeader_1.27mm:PinHeader_1x02_P1.27mm_Vertical, symbol Connector:Conn_01x02_Female
- added R5, R7: 10k, Resistor_SMD:R_0402_1005Metric, symbol Device:R
- added R8: RTERM, Resistor_SMD:R_0805_2012Metric_Pad1.20x1.40mm_HandSolder, symbol Device:R
- added RST1: TestPoint_Small, TestPoint:TestPoint_Pad_1.0x1.0mm, symbol Connector:TestPoint_Small
- added U1: ATmega4809-A, Package_QFP:TQFP-48_7x7mm_P0.5mm, symbol MCU_Microchip_ATmega:ATmega4809-A
- added U2: AMS1117-3.3, Package_TO_SOT_SMD:SOT-223-3_TabPin2, symbol Regulator_Linear:AMS1117-3.3
- added U3: SN65HVD75, Package_SO:SOIC-8_3.9x4.9mm_P1.27mm, symbol Interface_UART:SN65HVD75
- added U4, U5: 74HCT4051, Rare flowers:SOT763-1(DHVQFN16), symbol 74xx:74HCT4051
- C1: value 1uF/16V -> 10uF tant; footprint Capacitor_SMD:C_0402_1005Metric -> Capacitor_SMD:C_1206_3216Metric; JLC part number (none) -> C7171
- C2: value 1uF/6.3V -> 100uF tantalum; footprint Capacitor_SMD:C_0402_1005Metric -> Capacitor_SMD:C_1206_3216Metric; JLC part number (none) -> C16133
- C3, C4, C5, C6: JLC part number (none) -> C1525
- L1: JLC part number (none) -> C1035
- R1, R2, R6: value 10K -> 10k; JLC part number (none) -> C25744
- R3, R4: footprint Resistor_SMD:R_0603_1608Metric -> Resistor_SMD:R_1206_3216Metric; JLC part number (none) -> C17903
- TH1: Manufacturer part number (none) -> ERT-J0EG103JA; Mouser part number (none) -> 667-ERT-J0EG103JA
Connections:
- net RST is gone; now on net GND: R2.2
- net +3V3: now also C7.2, C8.2, J3.2 (VCC), U2.2 (VO), U3.8 (VCC), U4.16 (VCC), U5.16 (VCC); no longer C4.1
- net GND: now also C7.1, C8.1, J1.10 (Pin_10), J3.6 (GND), J4.8 (Pin_8), JPWR1.1 (Pin_1), R7.2, U1.15 (GND), U1.29 (GND), U1.43 (GND), U2.1 (GND), U3.5 (GND), U4.6 (~E), U4.7 (VEE), U4.8 (GND), U5.6 (~E), U5.7 (VEE), U5.8 (GND); no longer R6.1
- net RS485_A-: now also J1.7 (Pin_7), J4.11 (Pin_11), R8.2, RS4851.1 (Pin_1)
- net RS485_B+: now also J1.8 (Pin_8), J4.10 (Pin_10), R8.1, RS4851.2 (Pin_2)
- net RS485_EN: now also U1.46 (PA2), U3.2 (~RE), U3.3 (DE)
- net S0: now also U1.33 (PE3), U4.11 (S0)
- net S1: now also U1.32 (PE2), U4.10 (S1)
- net S2: now also U1.31 (PE1), U4.9 (S2)
- net UART_RX: now also U1.45 (PA1), U3.1 (RO)
- net UART_TX: now also U1.44 (PA0), U3.4 (DI)
- net Vin: now also J1.11 (Pin_11), J4.7 (Pin_7), JPWR1.2 (Pin_2), U2.3 (VI)
- net at C5.1, L1.2: now also C3.1, C4.1, R6.1, U1.14 (VCC), U1.28 (AVCC), U1.42 (VCC)
- net at R4.2: now also U3.7 (B)
- net at R3.2: now also U3.6 (A)
- net A_TOP: now reaches R2.1
- net A_TOP: now also U1.36 (PF2), U4.3 (A)
- net ADC renamed ADC_THERM
- net ADC_THERM: now also U1.27 (PD7)
- net Z: no longer names the net of R6.2
- net Z: now also R5.1
- new net: R5.2, RST1.1, U1.40 (PF6/~RESET)
- new net A: J4.9 (Pin_9), U1.47 (PA3)
- new net A-: J1.9 (Pin_9), U5.12 (A3)
- new net A_BOTTOM: R7.1, U1.23 (PD3), U5.3 (A)
- new net B: J4.6 (Pin_6), U4.13 (A0)
- new net B-: J1.6 (Pin_6), U1.13 (PC3)
- new net C: J4.5 (Pin_5), U1.39 (PF5)
- new net C-: J1.5 (Pin_5), U5.1 (A4)
- new net D: J4.4 (Pin_4), U4.12 (A3)
- new net D-: J1.4 (Pin_4), U1.8 (PB4)
- new net E: J4.3 (Pin_3), U1.38 (PF4)
- new net E-: J1.3 (Pin_3), U5.4 (A7)
- new net F: J4.2 (Pin_2), U4.5 (A5)
- new net F-: J1.2 (Pin_2), U1.7 (PB3)
- new net G: J4.1 (Pin_1), U1.37 (PF3)
- new net G-: J1.1 (Pin_1), U5.5 (A5)
- new net H: J4.12 (Pin_12), U4.14 (A1)
- new net H-: J1.12 (Pin_12), U1.24 (PD4)
- new net I: J4.13 (Pin_13), U1.48 (PA4)
- new net I-: J1.13 (Pin_13), U5.13 (A0)
- new net J: J4.14 (Pin_14), U4.15 (A2)
- new net J-: J1.14 (Pin_14), U1.25 (PD5)
- new net K: J4.15 (Pin_15), U1.1 (PA5)
- new net K-: J1.15 (Pin_15), U5.14 (A1)
- new net L: J4.16 (Pin_16), U4.1 (A4)
- new net L-: J1.16 (Pin_16), U1.26 (PD6)
- new net M: J4.17 (Pin_17), U1.2 (PA6)
- new net M-: J1.17 (Pin_17), U5.15 (A2)
- new net RXD: J3.4 (MOSI), U1.35 (PF1)
- new net S0-: U1.12 (PC2), U5.11 (S0)
- new net S1-: U1.11 (PC1), U5.10 (S1)
- new net S2-: U1.10 (PC0), U5.9 (S2)
- new net TXD: J3.5 (~RST), U1.34 (PF0)
- new net UPDI: J3.1 (MISO), U1.41 (UPDI)
- no-connect marks 96 -> 1
Other:
- note added: ".230W load at 20Mbps, 50% duty cycle test conditions (datasheet).\nresistors should be absolutely minimum rated to 1/4W\n(20Mbps is faster than we will be communicating, and we’re nowhere near 50% duty cycle for serial coms)."
- note added: "40mA GPIO sink/source current"
- note added: "A_BOTTOM to PD3 (A3 / AIN3)"
- note added: "A_TOP to PF2 (A12 / AIN12)"
- note added: "Half of the pins on the connector are for V+/0V, \nthe other half are for analog measurements."
- note added: "JLC actually stocks a smaller housing… but\ni already laid it out for SOIC-8, which makes\ntesting and troubleshooting easier anyway."
- note added: "On-chip IEC ESD protection is sufficient for laboratory and portable equipment but often insufficient for EFT and\nsurge transients occurring in industrial environments. Therefore, robust and reliable bus node design requires the\nuse of external transient protection devices."
- note added: "UPDI programming interface\n(for use with pogo pins, custom setup)"
- note added: "decoupling pins:\n14/15 28/29 42/43\n"
- note added: "output cap: larger the better \n(check LM1117 datasheet p.16)"
- note added: "test RS485 section\n"
- note added: "test points from serial port (uart)"
- moved on the sheet: C1, C2, C6, R1, R3, R4, TH1
