File: Schematics and PCBs/TFRAS_TOP/TFRAS_TOP.kicad_pcb (KiCad board)
At the start: 4 copper layers, 24 x 24 mm, 30 parts, among them J1 BOTTOM, J3 UPDI-POGO, J4 TOP, U1 ATmega4809-A, U2 AMS1117-3.3, U3 SN65HVD75, U4 74HCT4051, U5 74HCT4051

Commit message: PCB finished with seeed BOM
Parts:
- removed G***: LOGO, Rare flowers:TFRAS
- removed R5, R6: 10k, Resistor_SMD:R_0402_1005Metric
- added H1: logo, Rare flowers:TFRAS, B.Cu at (28.5, 24.3)
- C1: value 10u -> 10uF
- C2: value 100u -> 100uF
- R1: value 10k -> 100k
- R2: footprint Resistor_SMD:R_0402_1005Metric -> Resistor_SMD:R_0805_2012Metric; moved to B.Cu
- R3, R4: value 10 -> 13
- R7: footprint Resistor_SMD:R_0402_1005Metric -> Resistor_SMD:R_0805_2012Metric
- TH1: value Thermistor_NTC_10K -> Thermistor_NTC_100K; footprint Resistor_SMD:R_0402_1005Metric -> Resistor_SMD:R_0603_1608Metric
- U3: value SN65HVD75 -> MAX3471; footprint Package_SO:SOIC-8_3.9x4.9mm_P1.27mm -> Package_SO:MSOP-8_3x3mm_P0.65mm
- U4, U5: value 74HCT4051 -> 74HCT4051BQ
- moved R7 6.60 mm to (34.5, 42.8), turned to 0 degrees
- moved R2 4.47 mm to (41.8, 25.4), turned to 0 degrees
- moved R3 3.14 mm to (21.3, 34.1)
- moved R4 3.00 mm to (25.3, 34.1)
- moved U3 1.94 mm to (23.3, 29.9)
- moved R1 1.87 mm to (40.5, 36.5)
- moved RS4851 1.48 mm to (23.8, 36.9), turned to 90 degrees
- moved TH1 1.00 mm to (38.6, 36.0), turned to 270 degrees
- moved C6 0.81 mm to (21.6, 27.6)
Routing:
- net I-: track 14.5 -> 9.72 mm, vias 2 -> 1
- net GND: track 43.5 -> 38.7 mm, vias 14 -> 13
- net Net-(R4-Pad2): track 7.92 -> 5.38 mm
- net Net-(C3-Pad1): track 23.4 -> 21.3 mm, vias 3 -> 2
- net UART_RX: track 8.49 -> 6.60 mm
- net RS485_EN: track 9.25 -> 7.43 mm
- net ADC_THERM: track 3.20 -> 4.70 mm
- net A_TOP: track 16.9 -> 15.8 mm
- net +3V3: track 36.4 -> 35.3 mm, vias 8 -> 9
- net RS485_A-: track 33.1 -> 32.2 mm
- net Net-(R5-Pad1): track 0.89 -> 0.00 mm
- net UART_TX: track 10.7 -> 9.96 mm
- net RS485_B+: track 39.6 -> 39.0 mm
- net A_BOTTOM: track 17.6 -> 16.9 mm
Other:
- board text added: "-"
- board text removed: "V-"
