File: Schematics and PCBs/TFRAS_TOP/TFRAS_TOP.sch (KiCad schematic (older format))
At the start: 28 parts, among them J1 BOTTOM, J3 UPDI-POGO, J4 TOP, U1 ATmega4809-A, U2 AMS1117-3.3, U3 MAX3471, U4 74HC4051BQ, U5 74HC4051BQ

Commit message: tfras pcb
Other:
- note added: "REPLACE with MPM3610"
Changed lines of the file:
@@
 Text Notes 650  6750 0    50   ~ 0
 important note: it’s the HC version (3v3), not HCT (5v device)!
+Text Notes 450  -650 0    394  ~ 0
+REPLACE with  MPM3610
+Wire Notes Line
+	300  2350 3250 2350
+Wire Notes Line
+	3250 2350 3250 -450
+Wire Notes Line
+	3250 -450 300  -450
+Wire Notes Line
+	300  -450 300  2350
 $EndSCHEMATC
